Commit message: Clean up commit

File: assets/robot.xacro (robot description, xacro)
@@ -1,9 +1,6 @@
-<?xml version="1.0" ?>
-<!-- =================================================================================== -->
-<!-- |    This document was autogenerated by xacro from ur5_robotiq85_gripper.urdf.xacro | -->
-<!-- |    EDITING THIS FILE BY HAND IS NOT RECOMMENDED                                 | -->
-<!-- =================================================================================== -->
-<robot name="ur5">
-  <gazebo>
+<?xml version="1.0"?>
+<robot xmlns:xacro="http://www.ros.org/wiki/xacro" name="ur5">
+<xacro:arg name="path" default="/home/ubuntu20/gzweb_test/gzweb/http/client/assets/"/>
+<gazebo>
     <plugin filename="libgazebo_ros_control.so" name="ros_control">
       <!--robotNamespace>/</robotNamespace-->
@@ -30,5 +27,5 @@
       <origin rpy="0 0 3.141592653589793" xyz="0 0 0"/>
       <geometry>
-        <mesh filename="/home/ubuntu20/gzweb_test/gzweb/http/client/assets/ur_description/meshes/ur5/visual/base.dae"/>
+        <mesh filename="$(arg path)ur_description/meshes/ur5/visual/base.dae"/>
       </geometry>
       <material name="LightGrey">
@@ -39,5 +36,5 @@
       <origin rpy="0 0 3.141592653589793" xyz="0 0 0"/>
       <geometry>
-        <mesh filename="/home/ubuntu20/gzweb_test/gzweb/http/client/assets/ur_description/meshes/ur5/collision/base.stl"/>
+        <mesh filename="$(arg path)ur_description/meshes/ur5/collision/base.stl"/>
       </geometry>
     </collision>
@@ -60,5 +57,5 @@
       <origin rpy="0 0 3.141592653589793" xyz="0 0 0"/>
       <geometry>
-        <mesh filename="/home/ubuntu20/gzweb_test/gzweb/http/client/assets/ur_description/meshes/ur5/visual/shoulder.dae"/>
+        <mesh filename="$(arg path)ur_description/meshes/ur5/visual/shoulder.dae"/>
       </geometry>
       <material name="LightGrey">
@@ -69,5 +66,5 @@
       <origin rpy="0 0 3.141592653589793" xyz="0 0 0"/>
       <geometry>
-        <mesh filename="/home/ubuntu20/gzweb_test/gzweb/http/client/assets/ur_description/meshes/ur5/collision/shoulder.stl"/>
+        <mesh filename="$(arg path)ur_description/meshes/ur5/collision/shoulder.stl"/>
       </geometry>
     </collision>
@@ -90,5 +87,5 @@
       <origin rpy="1.5707963267948966 0 -1.5707963267948966" xyz="0 0 0.136"/>
       <geometry>
-        <mesh filename="/home/ubuntu20/gzweb_test/gzweb/http/client/assets/ur_description/meshes/ur5/visual/upperarm.dae"/>
+        <mesh filename="$(arg path)ur_description/meshes/ur5/visual/upperarm.dae"/>
       </geometry>
       <material name="LightGrey">
@@ -99,5 +96,5 @@
       <origin rpy="1.5707963267948966 0 -1.5707963267948966" xyz="0 0 0.136"/>
       <geometry>
-        <mesh filename="/home/ubuntu20/gzweb_test/gzweb/http/client/assets/ur_description/meshes/ur5/collision/upperarm.stl"/>
+        <mesh filename="$(arg path)ur_description/meshes/ur5/collision/upperarm.stl"/>
       </geometry>
     </collision>
@@ -120,5 +117,5 @@
       <origin rpy="1.5707963267948966 0 -1.5707963267948966" xyz="0 0 0.0165"/>
       <geometry>
-        <mesh filename="/home/ubuntu20/gzweb_test/gzweb/http/client/assets/ur_description/meshes/ur5/visual/forearm.dae"/>
+        <mesh filename="$(arg path)ur_description/meshes/ur5/visual/forearm.dae"/>
       </geometry>
       <material name="LightGrey">
@@ -129,5 +126,5 @@
       <origin rpy="1.5707963267948966 0 -1.5707963267948966" xyz="0 0 0.0165"/>
       <geometry>
-        <mesh filename="/home/ubuntu20/gzweb_test/gzweb/http/client/assets/ur_description/meshes/ur5/collision/forearm.stl"/>
+        <mesh filename="$(arg path)ur_description/meshes/ur5/collision/forearm.stl"/>
       </geometry>
     </collision>
@@ -150,5 +147,5 @@
       <origin rpy="1.5707963267948966 0 0" xyz="0 0 -0.093"/>
       <geometry>
-        <mesh filename="/home/ubuntu20/gzweb_test/gzweb/http/client/assets/ur_description/meshes/ur5/visual/wrist1.dae"/>
+        <mesh filename="$(arg path)ur_description/meshes/ur5/visual/wrist1.dae"/>
       </geometry>
       <material name="LightGrey">
@@ -159,5 +156,5 @@
       <origin rpy="1.5707963267948966 0 0" xyz="0 0 -0.093"/>
       <geometry>
-        <mesh filename="/home/ubuntu20/gzweb_test/gzweb/http/client/assets/ur_description/meshes/ur5/collision/wrist1.stl"/>
+        <mesh filename="$(arg path)ur_description/meshes/ur5/collision/wrist1.stl"/>
       </geometry>
     </collision>
@@ -180,5 +177,5 @@
       <origin rpy="0 0 0" xyz="0 0 -0.095"/>
       <geometry>
-        <mesh filename="/home/ubuntu20/gzweb_test/gzweb/http/client/assets/ur_description/meshes/ur5/visual/wrist2.dae"/>
+        <mesh filename="$(arg path)ur_description/meshes/ur5/visual/wrist2.dae"/>
       </geometry>
       <material name="LightGrey">
@@ -189,5 +186,5 @@
       <origin rpy="0 0 0" xyz="0 0 -0.095"/>
       <geometry>
-        <mesh filename="/home/ubuntu20/gzweb_test/gzweb/http/client/assets/ur_description/meshes/ur5/collision/wrist2.stl"/>
+        <mesh filename="$(arg path)ur_description/meshes/ur5/collision/wrist2.stl"/>
       </geometry>
     </collision>
@@ -210,5 +207,5 @@
       <origin rpy="1.5707963267948966 0 0" xyz="0 0 -0.0818"/>
       <geometry>
-        <mesh filename="/home/ubuntu20/gzweb_test/gzweb/http/client/assets/ur_description/meshes/ur5/visual/wrist3.dae"/>
+        <mesh filename="$(arg path)ur_description/meshes/ur5/visual/wrist3.dae"/>
       </geometry>
       <material name="LightGrey">
@@ -219,5 +216,5 @@
       <origin rpy="1.5707963267948966 0 0" xyz="0 0 -0.0823"/>
       <geometry>
-        <mesh filename="/home/ubuntu20/gzweb_test/gzweb/http/client/assets/ur_description/meshes/ur5/collision/wrist3.stl"/>
+        <mesh filename="$(arg path)ur_description/meshes/ur5/collision/wrist3.stl"/>
       </geometry>
     </collision>
@@ -346,5 +343,5 @@
     <visual>
       <geometry>
-        <mesh filename="/home/ubuntu20/gzweb_test/gzweb/http/client/assets/robotiq_description/meshes/robotiq_85_coupler.stl"/>
+        <mesh filename="$(arg path)robotiq_description/meshes/robotiq_85_coupler.stl"/>
       </geometry>
       <material name="flat_black"/>
@@ -352,5 +349,5 @@
     <collision>
       <geometry>
-        <mesh filename="/home/ubuntu20/gzweb_test/gzweb/http/client/assets/robotiq_description/meshes/robotiq_85_coupler.stl"/>
+        <mesh filename="$(arg path)robotiq_description/meshes/robotiq_85_coupler.stl"/>
       </geometry>
     </collision>
@@ -386,10 +383,10 @@
     <visual>
       <geometry>
-        <mesh filename="/home/ubuntu20/gzweb_test/gzweb/http/client/assets/robotiq_description/meshes/visual/robotiq_85_base_link.dae"/>
-      </geometry>
-    </visual>
-    <collision>
-      <geometry>
-        <mesh filename="/home/ubuntu20/gzweb_test/gzweb/http/client/assets/robotiq_description/meshes/collision/robotiq_85_base_link.stl"/>
+        <mesh filename="$(arg path)robotiq_description/meshes/visual/robotiq_85_base_link.dae"/>
+      </geometry>
+    </visual>
+    <collision>
+      <geometry>
+        <mesh filename="$(arg path)robotiq_description/meshes/collision/robotiq_85_base_link.stl"/>
       </geometry>
     </collision>
@@ -418,10 +415,10 @@
     <visual>
       <geometry>
-        <mesh filename="/home/ubuntu20/gzweb_test/gzweb/http/client/assets/robotiq_description/meshes/visual/robotiq_85_knuckle_link.dae"/>
-      </geometry>
-    </visual>
-    <collision>
-      <geometry>
-        <mesh filename="/home/ubuntu20/gzweb_test/gzweb/http/client/assets/robotiq_description/meshes/collision/robotiq_85_knuckle_link.stl"/>
+        <mesh filename="$(arg path)robotiq_description/meshes/visual/robotiq_85_knuckle_link.dae"/>
+      </geometry>
+    </visual>
+    <collision>
+      <geometry>
+        <mesh filename="$(arg path)robotiq_description/meshes/collision/robotiq_85_knuckle_link.stl"/>
       </geometry>
     </collision>
@@ -435,10 +432,10 @@
     <visual>
       <geometry>
-        <mesh filename="/home/ubuntu20/gzweb_test/gzweb/http/client/assets/robotiq_description/meshes/visual/robotiq_85_knuckle_link.dae"/>
-      </geometry>
-    </visual>
-    <collision>
-      <geometry>
-        <mesh filename="/home/ubuntu20/gzweb_test/gzweb/http/client/assets/robotiq_description/meshes/collision/robotiq_85_knuckle_link.stl"/>
+        <mesh filename="$(arg path)robotiq_description/meshes/visual/robotiq_85_knuckle_link.dae"/>
+      </geometry>
+    </visual>
+    <collision>
+      <geometry>
+        <mesh filename="$(arg path)robotiq_description/meshes/collision/robotiq_85_knuckle_link.stl"/>
       </geometry>
     </collision>
@@ -462,10 +459,10 @@
     <visual>
       <geometry>
-        <mesh filename="/home/ubuntu20/gzweb_test/gzweb/http/client/assets/robotiq_description/meshes/visual/robotiq_85_finger_link.dae"/>
-      </geometry>
-    </visual>
-    <collision>
-      <geometry>
-        <mesh filename="/home/ubuntu20/gzweb_test/gzweb/http/client/assets/robotiq_description/meshes/collision/robotiq_85_finger_link.stl"/>
+        <mesh filename="$(arg path)robotiq_description/meshes/visual/robotiq_85_finger_link.dae"/>
+      </geometry>
+    </visual>
+    <collision>
+      <geometry>
+        <mesh filename="$(arg path)robotiq_description/meshes/collision/robotiq_85_finger_link.stl"/>
       </geometry>
     </collision>
@@ -479,10 +476,10 @@
     <visual>
       <geometry>
-        <mesh filename="/home/ubuntu20/gzweb_test/gzweb/http/client/assets/robotiq_description/meshes/visual/robotiq_85_finger_link.dae"/>
-      </geometry>
-    </visual>
-    <collision>
-      <geometry>
-        <mesh filename="/home/ubuntu20/gzweb_test/gzweb/http/client/assets/robotiq_description/meshes/collision/robotiq_85_finger_link.stl"/>
+        <mesh filename="$(arg path)robotiq_description/meshes/visual/robotiq_85_finger_link.dae"/>
+      </geometry>
+    </visual>
+    <collision>
+      <geometry>
+        <mesh filename="$(arg path)robotiq_description/meshes/collision/robotiq_85_finger_link.stl"/>
       </geometry>
     </collision>
@@ -512,10 +509,10 @@
     <visual>
       <geometry>
-        <mesh filename="/home/ubuntu20/gzweb_test/gzweb/http/client/assets/robotiq_description/meshes/visual/robotiq_85_inner_knuckle_link.dae"/>
-      </geometry>
-    </visual>
-    <collision>
-      <geometry>
-        <mesh filename="/home/ubuntu20/gzweb_test/gzweb/http/client/assets/robotiq_description/meshes/collision/robotiq_85_inner_knuckle_link.stl"/>
+        <mesh filename="$(arg path)robotiq_description/meshes/visual/robotiq_85_inner_knuckle_link.dae"/>
+      </geometry>
+    </visual>
+    <collision>
+      <geometry>
+        <mesh filename="$(arg path)robotiq_description/meshes/collision/robotiq_85_inner_knuckle_link.stl"/>
       </geometry>
     </collision>
@@ -529,10 +526,10 @@
     <visual>
       <geometry>
-        <mesh filename="/home/ubuntu20/gzweb_test/gzweb/http/client/assets/robotiq_description/meshes/visual/robotiq_85_inner_knuckle_link.dae"/>
-      </geometry>
-    </visual>
-    <collision>
-      <geometry>
-        <mesh filename="/home/ubuntu20/gzweb_test/gzweb/http/client/assets/robotiq_description/meshes/collision/robotiq_85_inner_knuckle_link.stl"/>
+        <mesh filename="$(arg path)robotiq_description/meshes/visual/robotiq_85_inner_knuckle_link.dae"/>
+      </geometry>
+    </visual>
+    <collision>
+      <geometry>
+        <mesh filename="$(arg path)robotiq_description/meshes/collision/robotiq_85_inner_knuckle_link.stl"/>
       </geometry>
     </collision>
@@ -562,10 +559,10 @@
     <visual>
       <geometry>
-        <mesh filename="/home/ubuntu20/gzweb_test/gzweb/http/client/assets/robotiq_description/meshes/visual/robotiq_85_finger_tip_link.dae"/>
-      </geometry>
-    </visual>
-    <collision>
-      <geometry>
-        <mesh filename="/home/ubuntu20/gzweb_test/gzweb/http/client/assets/robotiq_description/meshes/collision/robotiq_85_finger_tip_link.stl"/>
+        <mesh filename="$(arg path)robotiq_description/meshes/visual/robotiq_85_finger_tip_link.dae"/>
+      </geometry>
+    </visual>
+    <collision>
+      <geometry>
+        <mesh filename="$(arg path)robotiq_description/meshes/collision/robotiq_85_finger_tip_link.stl"/>
       </geometry>
     </collision>
@@ -579,10 +576,10 @@
     <visual>
       <geometry>
-        <mesh filename="/home/ubuntu20/gzweb_test/gzweb/http/client/assets/robotiq_description/meshes/visual/robotiq_85_finger_tip_link.dae"/>
-      </geometry>
-    </visual>
-    <collision>
-      <geometry>
-        <mesh filename="/home/ubuntu20/gzweb_test/gzweb/http/client/assets/robotiq_description/meshes/collision/robotiq_85_finger_tip_link.stl"/>
+        <mesh filename="$(arg path)robotiq_description/meshes/visual/robotiq_85_finger_tip_link.dae"/>
+      </geometry>
+    </visual>
+    <collision>
+      <geometry>
+        <mesh filename="$(arg path)robotiq_description/meshes/collision/robotiq_85_finger_tip_link.stl"/>
       </geometry>
     </collision>
